File: EEPROM.sch (KiCad schematic (older format))
At the start: 22 parts, among them IC1 PCA6408APW, IC2 AT24CS01, U2 TPS613221ADBVT

Commit message: Assign schematic labels
Other:
- note added: "I2C peripherals"
Changed lines of the file:
@@
 Title "DDR5 testbed"
 Date "2022-03-02"
-Rev "1.0.0"
+Rev "1.0.1"
 Comp ""
 Comment1 ""
@@
 Text Label 6975 4450 0    50   ~ 0
 VDD_LED
+Text Notes 775  925  0    98   ~ 20
+I2C peripherals
 $EndSCHEMATC
