File: ddr5-testbed.sch (KiCad schematic (older format))
At the start: 2 parts

Commit message: Assign schematic labels
Changed lines of the file:
@@
 Title "DDR5 testbed"
 Date "2022-03-02"
-Rev "1.0.0"
+Rev "1.0.1"
 Comp ""
-Comment1 ""
-Comment2 ""
+Comment1 "www.antmicro.com"
+Comment2 "Antmicro Ltd."
 Comment3 ""
 Comment4 ""
 $EndDescr
 $Sheet
-S 6275 5275 1650 1125
+S 7650 5550 1650 1125
 U 5FDC4A05
 F0 "SODIMM" 50
@@
 DDR5 testbed
 $Sheet
-S 8625 5250 1650 1125
+S 10000 5525 1650 1125
 U 5FF943AC
 F0 "DDR5" 50
@@
 $EndComp
 $Sheet
-S 4000 5300 1600 1100
+S 5375 5575 1600 1100
 U 606DB5E6
 F0 "EEPROM" 50
