File: ddr5-testbed.kicad_sch (KiCad schematic)
At the start: 2 parts

Commit message: Globlib
Parts:
- N1: footprint ddr5-testbed-footprints:antmicro-logo_scaled_20mm -> antmicro-footprints:antmicro-logo; symbol ddr5-testbed:antmicro_logo -> antmicroMechanicalParts:antmicro_logo
- N2: footprint ddr5-testbed-footprints:oshw-logo -> antmicro-footprints:oshw-logo; symbol ddr5-testbed:oshw_logo -> antmicroMechanicalParts:oshw_logo
Changed lines of the file:
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@@
     (title "DDR5 testbed")
     (date "2023-01-13")
-    (rev "1.1.1")
+    (rev "1.1.1:8e7fe")
     (comment 1 "www.antmicro.com")
     (comment 2 "Antmicro Ltd.")
@@
     (effects (font (size 2.4892 2.4892) (thickness 0.4978) bold) (justify left bottom))
   )
-  (symbol (lib_id "ddr5-testbed:oshw_logo") (at 387.985 248.285 0) (unit 1)
+  (symbol (lib_id "antmicroMechanicalParts:oshw_logo") (at 387.985 248.285 0) (unit 1)
     (in_bom yes) (on_board yes) (dnp no) (fields_autoplaced)
     (property "Reference" "N2" (at 393.7 245.9925 0)
@@
       (effects (font (size 1.27 1.27) (thickness 0.15)) (justify left))
     )
-    (property "Footprint" "ddr5-testbed-footprints:oshw-logo" (at 403.225 258.445 0)
+    (property "Footprint" "antmicro-footprints:oshw-logo" (at 403.225 258.445 0)
       (effects (font (size 1.27 1.27) (thickness 0.15)) (justify left bottom) hide)
     )
@@
     )
   )
-  (symbol (lib_id "ddr5-testbed:antmicro_logo") (at 387.985 243.205 0) (unit 1)
+  (symbol (lib_id "antmicroMechanicalParts:antmicro_logo") (at 387.985 243.205 0) (unit 1)
     (in_bom yes) (on_board yes) (dnp no) (fields_autoplaced)
     (property "Reference" "N1" (at 393.7 240.9125 0)
@@
       (effects (font (size 1.27 1.27) (thickness 0.15)) (justify left))
     )
-    (property "Footprint" "ddr5-testbed-footprints:antmicro-logo_scaled_20mm" (at 403.225 253.365 0)
+    (property "Footprint" "antmicro-footprints:antmicro-logo" (at 403.225 253.365 0)
       (effects (font (size 1.27 1.27) (thickness 0.15)) (justify left bottom) hide)
     )

Commit message: Update footprints and symbols from library, clear DRC
Parts:
- N1: footprint antmicro-footprints:antmicro-logo -> antmicro-footprints:antmicro-logo_scaled_20mm
Changed lines of the file:
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@@
   (title_block
     (title "DDR5 testbed")
-    (date "2023-01-13")
-    (rev "1.1.1:9a23b")
+    (date "2024-05-27")
+    (rev "1.1.2")
     (comment 1 "www.antmicro.com")
     (comment 2 "Antmicro Ltd.")
@@
       (effects (font (size 1.27 1.27) (thickness 0.15)) (justify left))
     )
-    (property "Footprint" "antmicro-footprints:antmicro-logo" (at 403.225 253.365 0)
+    (property "Footprint" "antmicro-footprints:antmicro-logo_scaled_20mm" (at 403.225 253.365 0)
       (effects (font (size 1.27 1.27) (thickness 0.15)) (justify left bottom) hide)
     )
